Commit message: Adding Lidar and Camera

File: src/ros_mobile_robot/description/gazebo_control.xacro (robot description, xacro)
@@ -2,5 +2,5 @@
 <robot xmlns:xacro= "http://www.ros.org/wiki/xacro">
     <gazebo>
-        <plugin name="diff_drive" filename="libgazebo_ros_diffdrive.so">
+        <plugin name="diff_drive" filename="libgazebo_ros_diff_drive.so">
             <!-- Wheel Information-->
                 <left_joint>left_wheel_joint</left_joint>
@@ -15,5 +15,5 @@
                 <robot_base_frame>base_link</robot_base_frame>
                 <publish_odom>true</publish_odom>
-                <publish_odom_tf>tf</publish_odom_tf>
+                <publish_odom_tf>true</publish_odom_tf>
                 <publish_wheel_tf>true</publish_wheel_tf>
         </plugin>

File: src/ros_mobile_robot/description/robot.urdf.xacro (robot description, xacro)
@@ -3,3 +3,5 @@
     <xacro:include filename="robot_core.xacro"/>
     <xacro:include filename="gazebo_control.xacro"/>
+    <xacro:include filename="lidar.xacro"/>
+    <xacro:include filename="camera.xacro"/>
 </robot>

File: src/ros_mobile_robot/description/robot_core.xacro (robot description, xacro)
@@ -13,4 +13,7 @@
     <material name="blue">
         <color rgba="0 0 1 1"/>
+    </material>
+    <material name="red">
+        <color rgba="1 0 0 1"/>
     </material>
     <!-- Base-Link-->
@@ -124,4 +127,6 @@
         <gazebo reference = "caster_wheel_link">
             <material>Gazebo/Black</material>
+            <mu1 value = "0.05"/>
+            <mu2 value = "0.05"/>
          </gazebo>
 </robot>
